Commit message: Finished Rtab and communication bud was fixed.

File: urdf_try_1/urdf/urdf_try_1.xacro (robot description, xacro)
@@ -10,17 +10,17 @@
         <parent link="base_link"/>
         <child link="laser"/>
-        <origin xyz="0.0 0.0 0.1" rpy="0 0 0"/>
-    </joint>
-    <link name="base_footprint"/>
-    <joint name="base_joint" type="fixed">
-        <parent link="base_footprint"/>
-        <child link="base_link"/>
-        <origin xyz="0.0 0.0 0.01" rpy="0 0 0"/>
-    </joint>
+        <origin xyz="0.12 0.0 0.1" rpy="0 0 3.14"/>
+    </joint>
+<!--    <link name="base_footprint"/>-->
+<!--    <joint name="base_joint" type="fixed">-->
+<!--        <parent link="base_footprint"/>-->
+<!--        <child link="base_link"/>-->
+<!--        <origin xyz="0.0 0.0 0.01" rpy="0 0 0"/>-->
+<!--    </joint>-->
     <link
             name="base_link">
         <inertial>
             <origin
-                    xyz="0.115060400545944 -0.115447922845765 -0.0025"
+                    xyz="0 0 0"
                     rpy="0 0 0"/>
             <mass
